File: semana-06/projeto-instrução/projeto-instrução.kicad_pcb (KiCad board)
At the start: 2 copper layers, 7 parts, among them K1 Relay_SPDT, Q1 BC107, U1 Pico

Commit message: Ponderada Kicad
Parts:
- moved D1 51.3 mm to (82.5, 42.0)
- moved R1 43.7 mm to (83.7, 56.5)
- moved R2 41.8 mm to (98.4, 79.0)
- moved Q1 41.6 mm to (108.5, 78.0)
- moved K1 36.0 mm to (111.0, 51.0)
- moved D2 34.5 mm to (86.5, 71.5)
- moved U1 21.7 mm to (50.0, 65.5)
Routing:
- net saida_led: track 109.4 -> 33.2 mm
- net VCC: track 83.2 -> 146.9 mm
- net GND: track 84.4 -> 62.6 mm
- net sinal: track 57.6 -> 39.9 mm
- net Net-(D2-K): track 34.3 -> 19.3 mm
- net Net-(Q1-B): track 16.7 -> 10.5 mm
- net Net-(D1-A): track 46.2 -> 52.3 mm
